File: solenoid_driver/compact.kicad_sch (KiCad schematic)
At the start: 22 parts, among them J1 Conn_01x02, J2 Conn_01x02, J3 Conn_01x04, J4 Conn_01x02, Q1 IRLZ34N, Q2 IRLZ34N, U1 LM358, U2 L7805

Commit message: Add fan header to solenoid driver PCB
Parts:
- added J5: Conn_01x03, Connector_Molex:Molex_KK-254_AE-6410-03A_1x03_P2.54mm_Vertical, symbol Connector_Generic:Conn_01x03
Connections:
- net +12V: now also J5.2 (Pin_2)
- net GND: now also J5.1 (Pin_1)
- no-connect marks 0 -> 1
Other:
- moved on the sheet: U1C
